File: Teensy4.0-PCB/Teensy4.0/Teensy4.0.kicad_sch (KiCad schematic)
At the start: 74 parts, among them IC2 NC7WZ241K8X, J1 24-27, J2 28-31, U1 Teensy4.0, U2 Ai-Thinker-Ra-02, U3 TXS0104ERGYR, U4 TPS62143RGTT, U5 MIC5504-1.8YM5, U6 ICM-20948, U7 TXS0104ERGYR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

Commit message: updated some stuff
Changed lines of the file:
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@@
 (kicad_sch
-	(version 20231120)
+	(version 20250114)
 	(generator "eeschema")
-	(generator_version "8.0")
+	(generator_version "9.0")
 	(paper "A3")
 	(title_block
@@
 		(rev "V0.2")
 	)
+	(text "VCC -> 5V Buck Converter"
+		(exclude_from_sim no)
+		(at 76.454 218.186 0)
+		(effects
+			(font
+				(size 3.81 3.81)
+				(thickness 0.762)
+				(bold yes)
+			)
+		)
+	)
+	(text "JIRAKORN SUKMEE"
+		(exclude_from_sim no)
+		(at 351.79 262.128 0)
+		(effects
+			(font
+				(face "KiCad Font")
+				(size 5.08 5.08)
+				(thickness 1.016)
+				(bold yes)
+				(italic yes)
+				(color 0 0 0 1)
+			)
+		)
+	)
+	(text "IMU BIDIRECTIONAL\nLOGIC CONVERTER\n1V8 <-> 3V3"
+		(exclude_from_sim no)
+		(at 68.326 137.922 0)
+		(effects
+			(font
+				(size 3.048 3.048)
+				(thickness 0.762)
+				(bold yes)
+			)
+		)
+	)
+	(text "Button and Buzzer circuit"
+		(exclude_from_sim no)
+		(at 331.216 115.824 0)
+		(effects
+			(font
+				(size 3.048 3.048)
+				(thickness 0.762)
+				(bold yes)
+			)
+		)
+	)
+	(text "LoRa RA-02\nModule\n"
+		(exclude_from_sim no)
+		(at 304.8 50.038 0)
+		(effects
+			(font
+				(size 3.048 3.048)
+				(thickness 0.762)
+				(bold yes)
+			)
+		)
+	)
+	(text "Main Power\nBulk Capacitor\nMounting Holes"
+		(exclude_from_sim no)
+		(at 377.19 50.8 0)
+		(effects
+			(font
+				(size 3.048 3.048)
+				(thickness 0.762)
+				(bold yes)
+			)
+		)
+	)
+	(text "should work?"
+		(exclude_from_sim no)
+		(at 325.628 128.016 0)
+		(effects
+			(font
+				(size 2.54 2.54)
+				(thickness 0.508)
+				(bold yes)
+				(color 255 0 0 1)
+			)
+		)
+	)
+	(text "Green\n"
+		(exclude_from_sim no)
+		(at 400.304 94.996 0)
+		(effects
+			(font
+				(size 1.27 1.27)
+				(color 0 132 0 1)
+			)
+		)
+	)
+	(text "SERVO\nCONNECTIONS\n\n"
+		(exclude_from_sim no)
+		(at 319.278 190.5 0)
+		(effects
+			(font
+				(size 3.048 3.048)
+				(thickness 0.762)
+				(bold yes)
+			)
+		)
+	)
+	(text "ICM-20948 IMU\n"
+		(exclude_from_sim no)
+		(at 130.81 140.716 0)
+		(effects
+			(font
+				(size 3.048 3.048)
+				(thickness 0.762)
+				(bold yes)
+			)
+		)
+	)
+	(text "5V -> 1V8 LDO and power LED\n"
+		(exclude_from_sim no)
+		(at 255.016 162.814 0)
+		(effects
+			(font
+				(size 3.048 3.048)
+				(thickness 0.762)
+				(bold yes)
+			)
+		)
+	)
+	(text "SERVO LOGIC CONVERTER\n"
+		(exclude_from_sim no)
+		(at 216.408 220.472 0)
+		(effects
+			(font
+				(size 3.81 3.81)
+				(thickness 0.762)
+				(bold yes)
+			)
+		)
+	)
 	(junction
 		(at 87.63 152.4)
@@
 		)
 	)
-	(text "VCC -> 5V Buck Converter"
-		(exclude_from_sim no)
-		(at 76.454 218.186 0)
-		(effects
-			(font
-				(size 3.81 3.81)
-				(thickness 0.762)
-				(bold yes)
-			)
-		)
-	)
-	(text "JIRAKORN SUKMEE"
-		(exclude_from_sim no)
-		(at 351.79 262.128 0)
-		(effects
-			(font
-				(face "KiCad Font")
-				(size 5.08 5.08)
-				(thickness 1.016)
-				(bold yes)
-				(italic yes)
-				(color 0 0 0 1)
-			)
-		)
-	)
-	(text "IMU BIDIRECTIONAL\nLOGIC CONVERTER\n1V8 <-> 3V3"
-		(exclude_from_sim no)
-		(at 68.326 137.922 0)
-		(effects
-			(font
-				(size 3.048 3.048)
-				(thickness 0.762)
-				(bold yes)
-			)
-		)
-	)
-	(text "Button and Buzzer circuit"
-		(exclude_from_sim no)
-		(at 331.216 115.824 0)
-		(effects
-			(font
-				(size 3.048 3.048)
-				(thickness 0.762)
-				(bold yes)
-			)
-		)
-	)
-	(text "LoRa RA-02\nModule\n"
-		(exclude_from_sim no)
-		(at 304.8 50.038 0)
-		(effects
-			(font
-				(size 3.048 3.048)
-				(thickness 0.762)
-				(bold yes)
-			)
-		)
-	)
-	(text "Main Power\nBulk Capacitor\nMounting Holes"
-		(exclude_from_sim no)
-		(at 377.19 50.8 0)
-		(effects
-			(font
-				(size 3.048 3.048)
-				(thickness 0.762)
-				(bold yes)
-			)
-		)
-	)
-	(text "should work?"
-		(exclude_from_sim no)
-		(at 325.628 128.016 0)
-		(effects
-			(font
-				(size 2.54 2.54)
-				(thickness 0.508)
-				(bold yes)
-				(color 255 0 0 1)
-			)
-		)
-	)
-	(text "Green\n"
-		(exclude_from_sim no)
-		(at 400.304 94.996 0)
-		(effects
-			(font
-				(size 1.27 1.27)
-				(color 0 132 0 1)
-			)
-		)
-	)
-	(text "SERVO\nCONNECTIONS\n\n"
-		(exclude_from_sim no)
-		(at 319.278 190.5 0)
-		(effects
-			(font
-				(size 3.048 3.048)
-				(thickness 0.762)
-				(bold yes)
-			)
-		)
-	)
-	(text "ICM-20948 IMU\n"
-		(exclude_from_sim no)
-		(at 130.81 140.716 0)
-		(effects
-			(font
-				(size 3.048 3.048)
-				(thickness 0.762)
-				(bold yes)
-			)
-		)
-	)
-	(text "5V -> 1V8 LDO and power LED\n"
-		(exclude_from_sim no)
-		(at 255.016 162.814 0)
-		(effects
-			(font
-				(size 3.048 3.048)
-				(thickness 0.762)
-				(bold yes)
-			)
-		)
-	)
-	(text "SERVO LOGIC CONVERTER\n"
-		(exclude_from_sim no)
-		(at 216.408 220.472 0)
-		(effects
-			(font
-				(size 3.81 3.81)
-				(thickness 0.762)
-				(bold yes)
-			)
-		)
-	)
 	(label "serial_tx3"
 		(at 62.23 69.85 180)
@@
 		)
 	)
+	(embedded_fonts no)
 )
